File: PCB/Controller/Controller.kicad_sch (KiCad schematic)
At the start: 0 parts

Commit message: Update
Parts:
- added CN1: XT60PW_M, lcsc:CONN-TH_XT60PW-M, symbol LCSC:XT60PW-M
- added CN2: XT60PW_F, lcsc:TH_2P-XT60PW-F, symbol LCSC:XT60PW-F_C428722
- added CN3: Camera Conn, lcsc:CONN-TH_S3B-ZR-SM4A-TF-LF-SN, symbol LCSC:S3B-ZR-SM4A-TF(LF)(SN)
- added Card1: SD-006M, LCSC:SD-SMD_SD-006M, symbol LCSC:SD-006M
- added J1: Screw_Terminal_01x02, symbol Connector:Screw_Terminal_01x02
- added LED1: FJ2481CH, LCSC:LED-SEG-TH_14P-L32.2-W10.2-P2.54-S7.62-BL, symbol LCSC:FJ2481CH
- added R1, R2: 5.1K, symbol Device:R
- added SW1: TS-1088-AR02016, lcsc:SW-SMD_L3.9-W3.0-P4.45, symbol LCSC:TS-1088-AR02016
- added U1: STM32F765VGTx, Package_QFP:LQFP-100_14x14mm_P0.5mm, symbol MCU_ST_STM32F7:STM32F765VGTx
- added U10: BQ40Z50RSMR-R2, LCSC:VQFN-32_L4.0-W4.0-P0.40-TL-EP1.4_2, symbol LCSC:BQ40Z50RSMR-R2
- added U11: INA226AQDGSRQ1, LCSC:VSSOP-10_L3.0-W3.0-P0.50-LS4.9-BL, symbol LCSC:INA226AQDGSRQ1
- added U12: LMR51430, Package_TO_SOT_SMD:SOT-23-6, symbol Regulator_Switching:LMR51430
- added U2: BNO080, LCSC:LGA-28_L5.2-W3.8-P0.50-BL-1, symbol LCSC:BNO080
- added U3: BMP580, LCSC:LGA-10_L2.0-W2.0-P0.50-TL_BMP580, symbol LCSC:BMP580
- added U4: BQ25703ARSNR, LCSC:VQFN-32_L4.0-W4.0-P0.40-TL-EP, symbol LCSC:BQ25703ARSNR
- added U5: MAX7456EUI, LCSC:HTSSOP-28_L9.7-W4.4-P0.65-LS6.4-BL-EP5.5, symbol LCSC:MAX7456EUI
- added U6: SMA_Conn, lcsc:SMA-TH_SMA-KWE_C7498154, symbol LCSC:SMA-KWE_C7498154
- added U7: AL8871QT16E-13, LCSC:TSSOP-16_L5.0-W4.4-P0.65-LS6.4-BL-EP-2, symbol LCSC:AL8871QT16E-13
- added U8: STUSB4500QTR, Package_DFN_QFN:QFN-24-1EP_4x4mm_P0.5mm_EP2.7x2.7mm, symbol Interface_USB:STUSB4500QTR
- added U9: TPS630701RNMT, LCSC:VQFN-15_L3.0-W2.5-P0.50-BL, symbol LCSC:TPS630701RNMT
- added USB1: TYPE-C 16P(073), lcsc:USB-C-SMD_TYPE-C16PIN_C668624, symbol LCSC:TYPE-C16P(073)
Connections:
- new net: U1.10 (VSS), U1.26 (VSS), U1.49 (VSS), U1.74 (VSS), U1.99 (VSS)
- new net: U8.10 (GND), U8.25 (GND)
- new net: R2.1, USB1.A5 (CC1)
- new net: R1.1, USB1.B5 (CC2)
- new net GND: R1.2, R2.2, USB1.1 (SHELL), USB1.2 (SHELL), USB1.3 (SHELL), USB1.4 (SHELL), USB1.A1B12 (GND), USB1.B1A12 (GND)
- new net USB_DN: USB1.A7 (DN1), USB1.B7 (DN2)
- new net USB_DP: USB1.A6 (DP1), USB1.B6 (DP2)
- new net VBUS: USB1.A4B9 (VBUS), USB1.B4A9 (VBUS)
- no-connect marks 0 -> 2
